File: dombrick45.kicad_pcb (KiCad board)
At the start: 2 copper layers, 77 x 38.1 mm, 24 parts, among them SW1 SW_Push, U1 ATmega32U4-AU, Y1 16MHz

Commit message: 2019-10-06 tutorial
hobo kansei
Parts:
- moved C7 7.49 mm to (80.9, 96.6), turned to 270 degrees
- turned R1 to 90 degrees
Connections:
- U1 pad 27: Net-(U1-Pad27) -> ROW0
- U1 pad 28: Net-(U1-Pad28) -> COL1
- U1 pad 29: Net-(U1-Pad29) -> COL0
- U1 pad 30: Net-(U1-Pad30) -> ROW1
Routing:
- net COL1: track 19.1 -> 53.5 mm
- net ROW1: track 20.1 -> 52.8 mm
- net GND: track 107.6 -> 139.9 mm
- net ROW0: track 20.6 -> 48.3 mm
- net COL0: track 18.1 -> 33.8 mm
- net Net-(R1-Pad1): track 20.0 -> 30.8 mm
- net +5V: track 92.1 -> 98.9 mm

Commit message: 2019-10-06 tutorial last
Routing:
- net GND: track 139.9 -> 142.3 mm
- added copper zone on B.Cu, net GND
Other:
- board text added: "Dombrick45 starts here…."

Commit message: dombrick45 sematic to pcb tochuu
Parts:
- added D10: SOD-123, Diode_SMD:D_SOD-123, B.Cu at (212.7, 41.3)
- added D11: SOD-123, Diode_SMD:D_SOD-123, B.Cu at (231.8, 41.3)
- added D12: SOD-123, Diode_SMD:D_SOD-123, B.Cu at (250.8, 41.3)
- added D13: SOD-123, Diode_SMD:D_SOD-123, B.Cu at (273.1, 41.3)
- added D16: SOD-123, Diode_SMD:D_SOD-123, B.Cu at (84.1, 60.3)
- added D17: SOD-123, Diode_SMD:D_SOD-123, B.Cu at (103.2, 60.6)
- added D18: SOD-123, Diode_SMD:D_SOD-123, B.Cu at (122.2, 60.3)
- added D19: SOD-123, Diode_SMD:D_SOD-123, B.Cu at (141.3, 60.2)
- added D20: SOD-123, Diode_SMD:D_SOD-123, B.Cu at (160.3, 60.1)
- added D21: SOD-123, Diode_SMD:D_SOD-123, B.Cu at (179.4, 60.3)
- added D22: SOD-123, Diode_SMD:D_SOD-123, B.Cu at (198.4, 60.3)
- added D23: SOD-123, Diode_SMD:D_SOD-123, B.Cu at (217.5, 60.3)
- added D24: SOD-123, Diode_SMD:D_SOD-123, B.Cu at (236.5, 60.4)
- added D25: SOD-123, Diode_SMD:D_SOD-123, B.Cu at (255.6, 60.4)
- added D26: SOD-123, Diode_SMD:D_SOD-123, B.Cu at (274.6, 60.3)
- added D27: SOD-123, Diode_SMD:D_SOD-123, B.Cu at (54.8, 79.1)
- added D28: SOD-123, Diode_SMD:D_SOD-123, B.Cu at (74.6, 79.4)
- added D29: SOD-123, Diode_SMD:D_SOD-123, B.Cu at (93.8, 79.4)
- added D3: SOD-123, Diode_SMD:D_SOD-123, B.Cu at (79.4, 41.3)
- added D30: SOD-123, Diode_SMD:D_SOD-123, B.Cu at (112.7, 79.4)
- added D31: SOD-123, Diode_SMD:D_SOD-123, B.Cu at (131.8, 79.4)
- added D32: SOD-123, Diode_SMD:D_SOD-123, B.Cu at (150.7, 79.4)
- added D33: SOD-123, Diode_SMD:D_SOD-123, B.Cu at (169.9, 79.4)
- added D34: SOD-123, Diode_SMD:D_SOD-123, B.Cu at (188.9, 79.4)
- added D35: SOD-123, Diode_SMD:D_SOD-123, B.Cu at (208.0, 79.4)
- added D36: SOD-123, Diode_SMD:D_SOD-123, B.Cu at (227.0, 79.4)
- added D37: SOD-123, Diode_SMD:D_SOD-123, B.Cu at (246.1, 79.4)
- added D38: SOD-123, Diode_SMD:D_SOD-123, B.Cu at (265.1, 78.6)
- added D39: SOD-123, Diode_SMD:D_SOD-123, B.Cu at (46.0, 98.6)
- added D4: SOD-123, Diode_SMD:D_SOD-123, B.Cu at (98.4, 41.5)
- added D40: SOD-123, Diode_SMD:D_SOD-123, B.Cu at (65.1, 98.4)
- added D41: SOD-123, Diode_SMD:D_SOD-123, B.Cu at (87.3, 98.4)
- added D42: SOD-123, Diode_SMD:D_SOD-123, B.Cu at (111.9, 98.4)
- added D43: SOD-123, Diode_SMD:D_SOD-123, B.Cu at (135.7, 98.4)
- added D44: SOD-123, Diode_SMD:D_SOD-123, B.Cu at (184.2, 97.6)
- added D45: SOD-123, Diode_SMD:D_SOD-123, B.Cu at (211.9, 98.4)
- added D46: SOD-123, Diode_SMD:D_SOD-123, B.Cu at (231.8, 98.4)
- added D47: SOD-123, Diode_SMD:D_SOD-123, B.Cu at (250.8, 98.4)
- added D48: SOD-123, Diode_SMD:D_SOD-123, B.Cu at (269.9, 98.4)
- added D5: SOD-123, Diode_SMD:D_SOD-123, B.Cu at (117.0, 41.4)
- added D6: SOD-123, Diode_SMD:D_SOD-123, B.Cu at (136.8, 41.0)
- added D7: SOD-123, Diode_SMD:D_SOD-123, B.Cu at (155.2, 41.2)
- added D8: SOD-123, Diode_SMD:D_SOD-123, B.Cu at (174.2, 41.2)
- added D9: SOD-123, Diode_SMD:D_SOD-123, B.Cu at (193.7, 41.6)
- added MX10: MX-NoLED, MX_Alps_Hybrid:MX-1U-NoLED, F.Cu at (204.8, 41.3)
- added MX11: MX-NoLED, MX_Alps_Hybrid:MX-1U-NoLED, F.Cu at (223.8, 41.4)
- added MX12: MX-NoLED, MX_Alps_Hybrid:MX-1U-NoLED, F.Cu at (242.9, 41.3)
- added MX13: MX-NoLED, MX_Alps_Hybrid:MX-1.25U-NoLED, F.Cu at (264.3, 41.3)
- added MX16: MX-NoLED, MX_Alps_Hybrid:MX-1U-NoLED, F.Cu at (76.2, 60.3)
- added MX17: MX-NoLED, MX_Alps_Hybrid:MX-1U-NoLED, F.Cu at (95.2, 60.3)
- added MX18: MX-NoLED, MX_Alps_Hybrid:MX-1U-NoLED, F.Cu at (114.3, 60.3)
- added MX19: MX-NoLED, MX_Alps_Hybrid:MX-1U-NoLED, F.Cu at (133.3, 60.3)
- added MX20: MX-NoLED, MX_Alps_Hybrid:MX-1U-NoLED, F.Cu at (152.4, 60.3)
- added MX21: MX-NoLED, MX_Alps_Hybrid:MX-1U-NoLED, F.Cu at (171.4, 60.3)
- added MX22: MX-NoLED, MX_Alps_Hybrid:MX-1U-NoLED, F.Cu at (190.5, 60.3)
- added MX23: MX-NoLED, MX_Alps_Hybrid:MX-1U-NoLED, F.Cu at (209.6, 60.3)
- added MX24: MX-NoLED, MX_Alps_Hybrid:MX-1U-NoLED, F.Cu at (228.6, 60.3)
- added MX25: MX-NoLED, MX_Alps_Hybrid:MX-1U-NoLED, F.Cu at (247.7, 60.3)
- added MX26: MX-NoLED, MX_Alps_Hybrid:MX-1U-NoLED, F.Cu at (266.7, 60.3)
- added MX27: MX-NoLED, MX_Alps_Hybrid:MX-1.25U-NoLED, F.Cu at (45.2, 79.4)
- added MX28: MX-NoLED, MX_Alps_Hybrid:MX-1U-NoLED, F.Cu at (66.7, 79.4)
- added MX29: MX-NoLED, MX_Alps_Hybrid:MX-1U-NoLED, F.Cu at (85.7, 79.4)
- added MX3: MX-NoLED, MX_Alps_Hybrid:MX-1U-NoLED, F.Cu at (71.4, 41.3)
- added MX30: MX-NoLED, MX_Alps_Hybrid:MX-1U-NoLED, F.Cu at (104.8, 79.4)
- added MX31: MX-NoLED, MX_Alps_Hybrid:MX-1U-NoLED, F.Cu at (123.8, 79.4)
- added MX32: MX-NoLED, MX_Alps_Hybrid:MX-1U-NoLED, F.Cu at (142.8, 79.4)
- added MX33: MX-NoLED, MX_Alps_Hybrid:MX-1U-NoLED, F.Cu at (161.9, 79.4)
- added MX34: MX-NoLED, MX_Alps_Hybrid:MX-1U-NoLED, F.Cu at (181.0, 79.4)
- added MX35: MX-NoLED, MX_Alps_Hybrid:MX-1U-NoLED, F.Cu at (200.0, 79.4)
- added MX36: MX-NoLED, MX_Alps_Hybrid:MX-1U-NoLED, F.Cu at (219.1, 79.4)
- added MX37: MX-NoLED, MX_Alps_Hybrid:MX-1U-NoLED, F.Cu at (238.1, 79.4)
- added MX38: MX-NoLED, MX_Alps_Hybrid:MX-1U-NoLED, F.Cu at (257.2, 79.4)
- added MX39: MX-NoLED, MX_Alps_Hybrid:MX-1U-NoLED, F.Cu at (38.1, 98.4)
- added MX4: MX-NoLED, MX_Alps_Hybrid:MX-1U-NoLED, F.Cu at (90.5, 41.3)
- added MX40: MX-NoLED, MX_Alps_Hybrid:MX-1U-NoLED, F.Cu at (57.1, 98.4)
- added MX41: MX-NoLED, MX_Alps_Hybrid:MX-1.25U-NoLED, F.Cu at (78.6, 98.4)
- added MX42: MX-NoLED, MX_Alps_Hybrid:MX-1.25U-NoLED, F.Cu at (102.2, 98.6)
- added MX43: MX-NoLED, MX_Alps_Hybrid:MX-1.25U-NoLED, F.Cu at (126.2, 98.4)
- added MX44: MX-NoLED, MX_Alps_Hybrid:MX-2.75U-NoLED, F.Cu at (164.3, 98.4)
- added MX45: MX-NoLED, MX_Alps_Hybrid:MX-1.25U-NoLED, F.Cu at (202.4, 98.4)
- added MX46: MX-NoLED, MX_Alps_Hybrid:MX-1U-NoLED, F.Cu at (223.8, 98.4)
- added MX47: MX-NoLED, MX_Alps_Hybrid:MX-1U-NoLED, F.Cu at (242.9, 98.4)
- added MX48: MX-NoLED, MX_Alps_Hybrid:MX-1U-NoLED, F.Cu at (261.9, 98.4)
- added MX5: MX-NoLED, MX_Alps_Hybrid:MX-1U-NoLED, F.Cu at (109.5, 41.3)
- added MX6: MX-NoLED, MX_Alps_Hybrid:MX-1U-NoLED, F.Cu at (128.6, 41.3)
- added MX7: MX-NoLED, MX_Alps_Hybrid:MX-1U-NoLED, F.Cu at (147.6, 41.3)
- added MX8: MX-NoLED, MX_Alps_Hybrid:MX-1U-NoLED, F.Cu at (166.7, 41.3)
- added MX9: MX-NoLED, MX_Alps_Hybrid:MX-1U-NoLED, F.Cu at (185.7, 41.3)
- MX14: renamed from MX3; footprint MX_Alps_Hybrid:MX-1U-NoLED -> MX_Alps_Hybrid:MX-1.25U-NoLED
- moved Y1 99.2 mm to (39.9, 164.8)
- moved C1 99.2 mm to (44.2, 164.8)
- moved C2 99.2 mm to (35.4, 164.8)
- moved C3 99.2 mm to (29.9, 177.2)
- moved C4 99.2 mm to (44.0, 187.1)
- moved C5 99.2 mm to (32.5, 169.0)
- moved C6 99.2 mm to (49.9, 173.6)
- moved C7 99.2 mm to (30.6, 182.1)
- moved F1 99.2 mm to (18.3, 174.6)
- moved R1 99.2 mm to (29.1, 169.1)
- moved R2 99.2 mm to (22.1, 169.0)
- moved R4 99.2 mm to (49.9, 182.5)
- moved SW1 99.2 mm to (21.6, 185.9)
- moved R3 99.2 mm to (19.2, 169.0)
- moved U1 99.2 mm to (40.2, 177.5)
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- renumbered D3 to D14, D4 to D15, MX4 to MX15
Routing:
- net COL1: track 53.5 -> 0.00 mm
- net ROW1: track 52.8 -> 0.00 mm
- net ROW0: track 48.3 -> 0.00 mm
- net COL0: track 33.8 -> 0.00 mm
- net Net-(D2-Pad2): track 6.64 -> 0.00 mm
- net Net-(D1-Pad2): track 6.64 -> 0.00 mm
- net Net-(D14-Pad2): track 6.62 -> 0.00 mm
- net Net-(D15-Pad2): track 6.62 -> 0.00 mm

Commit message: 2019-10-10 keysw connect
Parts:
- added MX49: MX-NoLED, MX_Only:MXOnly-6.25U-Hotswap, F.Cu at (150.0, 98.4)
- added MX50: MX-NoLED, MX_Only:MXOnly-1.25U-Hotswap, F.Cu at (221.5, 98.4)
- MX39, MX46, MX48: footprint MX_Alps_Hybrid:MX-1U-NoLED -> MX_Only:MXOnly-1U-Hotswap
- MX42, MX43, MX45: footprint MX_Alps_Hybrid:MX-1.25U-NoLED -> MX_Only:MXOnly-1.25U-Hotswap
- MX44: footprint MX_Alps_Hybrid:MX-2.75U-NoLED -> MX_Only:MXOnly-2.75U-Hotswap-ReversedStabilizers
- moved U1 65.7 mm to (88.1, 132.6), turned to 45 degrees
- moved USB1 16.6 mm to (23.0, 142.9)
- moved D1 15.8 mm to (27.8, 50.0)
- moved D44 11.9 mm to (172.2, 98.4)
- moved D2 9.06 mm to (58.7, 50.0)
- moved D46 6.35 mm to (231.8, 92.1)
- moved D33 6.29 mm to (169.9, 85.7)
- moved D45 5.67 mm to (212.7, 104.0), turned to 270 degrees
- moved D20 4.51 mm to (160.3, 55.6)
- moved D34 0.86 mm to (188.9, 78.6)
- moved MX42 0.22 mm to (102.4, 98.4)
- moved MX32 0.11 mm to (142.9, 79.4)
- turned MX1 to 180 degrees
- turned MX2 to 180 degrees
- turned MX33 to 180 degrees
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Connections:
- MX35 pad 1: Net-(MX35-Pad1) -> COL3
- MX36 pad 1: Net-(MX36-Pad1) -> COL2
- MX37 pad 1: Net-(MX37-Pad1) -> COL1
- MX44 pad 1: Net-(MX44-Pad1) -> COL4
- MX45 pad 1: Net-(MX35-Pad1) -> COL3
- MX46 pad 1: Net-(MX36-Pad1) -> COL2
- MX47 pad 1: Net-(MX37-Pad1) -> COL1
Routing:
- net COL0: track 0.00 -> 354.5 mm, vias 0 -> 4
- net COL1: track 0.00 -> 305.0 mm, vias 0 -> 2
- net COL2: track 0.00 -> 297.5 mm, vias 0 -> 4
- net COL3: track 0.00 -> 241.7 mm, vias 0 -> 4
- net COL4: track 0.00 -> 211.8 mm, vias 0 -> 4
- net ROW5: track 0.00 -> 135.3 mm
- net COL5: track 0.00 -> 131.7 mm
- net ROW4: track 0.00 -> 127.3 mm
- net ROW7: track 0.00 -> 125.4 mm
- net ROW0: track 0.00 -> 116.6 mm
- net ROW6: track 0.00 -> 105.5 mm
- net ROW1: track 0.00 -> 104.5 mm
- net ROW2: track 0.00 -> 103.5 mm
- net ROW3: track 0.00 -> 95.5 mm
- net Net-(D44-Pad2): track 0.00 -> 42.2 mm
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
Commit message: 2019-10-12 PBC ver0.1
Parts:
- moved F1 264.8 mm to (249.9, 46.4)
- moved R3 264.2 mm to (252.6, 45.1)
- moved R2 264.1 mm to (255.4, 45.1)
- moved USB1 256.0 mm to (254.4, 33.4)
- moved SW1 253.1 mm to (235.5, 50.6), turned to 0 degrees
- moved C3 243.3 mm to (244.8, 63.2), turned to 0 degrees
- moved C7 242.8 mm to (237.7, 55.5), turned to 180 degrees
- moved R1 240.5 mm to (246.6, 66.5)
- moved C5 240.4 mm to (249.6, 65.7)
- moved C2 239.1 mm to (253.4, 66.5)
- moved Y1 238.5 mm to (257.2, 66.5)
- moved C1 238.3 mm to (261.2, 66.5)
- moved C4 218.2 mm to (226.4, 67.3), turned to 90 degrees
- moved R4 208.7 mm to (224.0, 67.4), turned to 270 degrees
- moved C6 204.0 mm to (232.1, 81.9), turned to 0 degrees
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Connections:
- U1 pad 18: Net-(U1-Pad18) -> COL0
- U1 pad 19: Net-(U1-Pad19) -> ROW6
- U1 pad 20: Net-(U1-Pad20) -> ROW7
- U1 pad 21: Net-(U1-Pad21) -> COL1
- U1 pad 26: Net-(U1-Pad26) -> ROW3
- U1 pad 27: ROW0 -> ROW2
- U1 pad 28: COL1 -> COL5
- U1 pad 29: COL0 -> COL4
- U1 pad 30: ROW1 -> COL3
- U1 pad 31: Net-(U1-Pad31) -> COL2
- U1 pad 32: Net-(U1-Pad32) -> ROW1
- U1 pad 36: Net-(U1-Pad36) -> ROW0
- U1 pad 37: Net-(U1-Pad37) -> COL6
- U1 pad 38: Net-(U1-Pad38) -> ROW5
- U1 pad 39: Net-(U1-Pad39) -> ROW4
Routing:
- net ROW3: track 95.5 -> 231.9 mm
- net ROW0: track 116.6 -> 212.7 mm
- net ROW1: track 104.5 -> 198.2 mm
- net ROW2: track 103.5 -> 196.9 mm
- net COL6: track 21.0 -> 111.6 mm
- net COL5: track 131.7 -> 201.9 mm
- net COL4: track 211.8 -> 277.7 mm, vias 4 -> 3
- net ROW6: track 105.5 -> 157.9 mm, vias 0 -> 2
- net COL1: track 305.0 -> 351.6 mm, vias 2 -> 0
- net COL3: track 241.7 -> 282.5 mm, vias 4 -> 3
- net ROW5: track 135.3 -> 170.3 mm, vias 0 -> 2
- net COL0: track 354.5 -> 389.0 mm
- net ROW7: track 125.4 -> 150.2 mm, vias 0 -> 2
- net ROW4: track 127.3 -> 147.6 mm, vias 0 -> 4
- net COL2: track 297.5 -> 314.5 mm, vias 4 -> 2
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- removed copper zone on B.Cu, net GND
Other:
- board size 77 x 38.1 mm -> 252.4 x 76.2 mm

Commit message: 2019-10-12 haisen bishuusei
Routing:
- net GND: track 136.7 -> 135.0 mm

Commit message: 2019-10-12 advice itadaita ato
Parts:
- moved C1 16.2 mm to (248.0, 75.8), turned to 135 degrees
- moved Y1 9.31 mm to (250.7, 73.2), turned to 45 degrees
- moved R1 8.38 mm to (255.0, 66.3), turned to 180 degrees
- moved C2 4.03 mm to (253.3, 70.6), turned to 315 degrees
- moved R4 3.16 mm to (225.1, 70.4), turned to 0 degrees
- moved C4 1.49 mm to (225.0, 67.8), turned to 180 degrees
- moved C5 1.45 mm to (250.7, 66.5), turned to 0 degrees
- moved D25 0.95 mm to (255.6, 59.4)
Routing:
- net Net-(U1-Pad40): track 0.00 -> 16.7 mm
- net Net-(U1-Pad8): track 0.00 -> 16.3 mm
- net Net-(U1-Pad9): track 0.00 -> 15.6 mm
- net Net-(U1-Pad10): track 0.00 -> 15.1 mm
- net Net-(U1-Pad11): track 0.00 -> 14.6 mm
- net COL1: track 351.6 -> 364.2 mm
- net Net-(C1-Pad2): track 23.5 -> 12.3 mm
- net Net-(R1-Pad1): track 29.3 -> 39.8 mm, vias 2 -> 3
- net Net-(U1-Pad41): track 0.00 -> 6.72 mm
- net Net-(U1-Pad42): track 0.00 -> 6.19 mm
- net Net-(C2-Pad2): track 21.9 -> 17.4 mm
- net ROW5: track 170.3 -> 166.0 mm
- net Net-(R4-Pad2): track 7.63 -> 4.48 mm
- net +5V: track 114.8 -> 117.8 mm
- net Net-(U1-Pad25): track 0.00 -> 2.97 mm, vias 0 -> 1
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
Commit message: 2019-10-14 SPI toridashi and dombri mark
Parts:
- added J1: AVR-ISP-6, random-keyboard-parts:Reset_Pretty, B.Cu at (263.5, 67.3)
- MX40, MX47: footprint MX_Alps_Hybrid:MX-1U-NoLED -> MX_Only:MXOnly-1U-Hotswap
- MX41: footprint MX_Alps_Hybrid:MX-1.25U-NoLED -> MX_Only:MXOnly-1.25U-Hotswap
- moved D26 13.2 mm to (263.3, 52.8)
- moved D25 0.76 mm to (255.6, 58.7)
- moved R1 0.25 mm to (255.0, 66.5)
Connections:
- net Net-(R1-Pad1) renamed RESET
Routing:
- net RESET: track 39.8 -> 57.9 mm, vias 3 -> 4
- net Net-(J1-Pad4): track 15.1 -> 29.8 mm, vias 0 -> 1
- net +5V: track 117.8 -> 129.9 mm
- net GND: track 136.7 -> 148.7 mm
- net Net-(U1-Pad40): track 16.7 -> 7.86 mm, vias 0 -> 1
- net Net-(J1-Pad3): track 15.6 -> 24.2 mm
- net ROW5: track 166.0 -> 158.4 mm
- net Net-(U1-Pad8): track 16.3 -> 10.6 mm, vias 0 -> 1
- net Net-(J1-Pad1): track 14.6 -> 19.3 mm
- net Net-(D26-Pad2): track 10.0 -> 6.76 mm
- net ROW6: track 156.2 -> 153.2 mm
- net Net-(D41-Pad2): track 7.61 -> 4.71 mm
- net Net-(D40-Pad2): track 6.82 -> 4.31 mm
- net Net-(D47-Pad2): track 6.82 -> 4.31 mm
- net COL2: track 314.5 -> 316.5 mm, vias 2 -> 3
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Other:
- board text removed: "Dombrick45 starts here…."
