File: dombrick45.kicad_pcb (KiCad board)
At the start: 2 copper layers, 252.4 x 76.2 mm, 115 parts, among them J1 AVR-ISP-6, SW1 SW_Push, U1 ATmega32U4-AU, Y1 16MHz

Commit message: 2019-10-1
Other:
- board text added: "Dombrick45"

Commit message: 2019-10-21 usb-c impl, gnd filled and silk design completed.
Parts:
- added R5: 5.1k, Resistor_SMD:R_0805_2012Metric, B.Cu at (265.3, 45.3)
- added R6: 5.1k, Resistor_SMD:R_0805_2012Metric, B.Cu at (264.9, 51.8)
- added REF**: MountingHole_2.2mm_M2, MountingHole:MountingHole_2.2mm_M2, B.Cu at (263.3, 85.7)
- added REF**: MountingHole_2.2mm_M2, MountingHole:MountingHole_2.2mm_M2, B.Cu at (240.5, 45.7)
- added REF**: MountingHole_2.2mm_M2, MountingHole:MountingHole_2.2mm_M2, B.Cu at (157.1, 50.4)
- added REF**: MountingHole_2.2mm_M2, MountingHole:MountingHole_2.2mm_M2, B.Cu at (133.5, 85.2)
- added REF**: MountingHole_2.2mm_M2, MountingHole:MountingHole_2.2mm_M2, B.Cu at (56.0, 73.8)
- added REF**: MountingHole_2.2mm_M2, MountingHole:MountingHole_2.2mm_M2, B.Cu at (42.8, 50.2)
- added REF**: MountingHole_2.2mm_M2, MountingHole:MountingHole_2.2mm_M2, B.Cu at (233.2, 105.2)
- added REF**: MountingHole_2.2mm_M2, MountingHole:MountingHole_2.2mm_M2, B.Cu at (184.7, 92.2)
- added REF**: MountingHole_2.2mm_M2, MountingHole:MountingHole_2.2mm_M2, B.Cu at (68.1, 104.0)
- added U2: PRTR5V0U2X, random-keyboard-parts:SOT143B, B.Cu at (264.5, 48.7)
- added USB2: HRO-TYPE-C-31-M-12, Type-C:HRO-TYPE-C-31-M-12-Assembly, B.Cu at (277.0, 48.4)
- moved D13 16.0 mm to (272.9, 38.7), turned to 90 degrees
- moved D26 13.6 mm to (274.6, 60.3), turned to 90 degrees
- moved D48 6.11 mm to (269.9, 98.4), turned to 90 degrees
- moved D12 4.68 mm to (235.2, 41.4), turned to 90 degrees
- moved D37 4.44 mm to (244.6, 85.9)
- moved D24 3.45 mm to (222.5, 53.7), turned to 90 degrees
- moved SW1 3.30 mm to (232.2, 50.6)
- moved R2 1.53 mm to (254.8, 46.5)
- moved USB1 1.50 mm to (253.6, 34.7)
- moved R3 1.45 mm to (252.2, 46.5)
- moved F1 0.46 mm to (249.6, 46.6)
- turned D36 to 90 degrees
- turned D45 to 90 degrees
- turned MX12 to 0 degrees
- turned MX13 to 0 degrees
Routing:
- net GND: track 148.7 -> 178.0 mm, vias 0 -> 5
- net VCC: track 8.24 -> 35.6 mm, vias 0 -> 5
- net D+: track 6.72 -> 29.8 mm, vias 0 -> 2
- net ROW4: track 147.6 -> 168.7 mm, vias 4 -> 7
- net D-: track 6.70 -> 27.1 mm, vias 0 -> 2
- net COL1: track 365.5 -> 384.4 mm, vias 2 -> 3
- net ROW6: track 153.2 -> 143.6 mm
- net COL0: track 390.5 -> 400.0 mm
- net Net-(D48-Pad2): track 11.2 -> 4.06 mm
- net COL2: track 316.5 -> 321.3 mm
- net ROW7: track 151.0 -> 155.7 mm, vias 2 -> 4
- net ROW5: track 158.4 -> 163.1 mm
- net Net-(D12-Pad2): track 8.72 -> 13.2 mm
- net Net-(D37-Pad2): track 16.3 -> 11.8 mm
- net Net-(R6-Pad1): track 0.00 -> 4.29 mm
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- added copper zone on B.Cu, net GND
Other:
- board text added: "Dombrick45 : Dvorak Oriented 45% Keyboard"
- board text removed: "Dombrick45"

Commit message: 2019-10-22 hobo OK
Parts:
- removed REF** (x9): MountingHole_2.2mm_M2, MountingHole:MountingHole_2.2mm_M2
- added H1: MountingHole, MountingHole:MountingHole_2.2mm_M2, B.Cu at (42.8, 50.0)
- added H2: MountingHole, MountingHole:MountingHole_2.2mm_M2, B.Cu at (54.7, 73.4)
- added H3: MountingHole, MountingHole:MountingHole_2.2mm_M2, B.Cu at (158.5, 51.2)
- added H4: MountingHole, MountingHole:MountingHole_2.2mm_M2, B.Cu at (67.8, 103.9)
- added H5: MountingHole, MountingHole:MountingHole_2.2mm_M2, B.Cu at (242.2, 46.1)
- added H6: MountingHole, MountingHole:MountingHole_2.2mm_M2, B.Cu at (132.6, 85.1)
- added H7: MountingHole, MountingHole:MountingHole_2.2mm_M2, B.Cu at (185.5, 92.2)
- added H8: MountingHole, MountingHole:MountingHole_2.2mm_M2, B.Cu at (238.6, 104.8)
- added H9: MountingHole, MountingHole:MountingHole_2.2mm_M2, B.Cu at (263.5, 85.9)
- MX44: footprint MX_Only:MXOnly-2.75U-Hotswap-ReversedStabilizers -> MX_Only:MXOnly-2.75U-Hotswap
- MX49: footprint MX_Only:MXOnly-6.25U-Hotswap -> MX_Only:MXOnly-6.25U-Hotswap-ReversedStabilizers
- moved D44 3.84 mm to (176.0, 97.7)
- moved C6 1.19 mm to (231.8, 83.0), turned to 270 degrees
- moved C5 0.52 mm to (250.7, 67.1), turned to 270 degrees
- turned MX44 to 180 degrees
- turned MX45 to 0 degrees
- turned MX49 to 0 degrees
Routing:
- net COL1: track 384.4 -> 355.3 mm
- net COL4: track 277.2 -> 292.6 mm
- net ROW7: track 155.7 -> 145.0 mm, vias 4 -> 2
- net Net-(D45-Pad2): track 18.9 -> 11.0 mm
- net COL3: track 282.0 -> 274.9 mm
- net GND: track 178.0 -> 182.4 mm, vias 5 -> 6
- net Net-(D44-Pad2): track 42.2 -> 38.1 mm
- net ROW4: track 168.7 -> 165.8 mm, vias 7 -> 5
- net Net-(J1-Pad3): track 24.2 -> 25.5 mm
- net Net-(J1-Pad4): track 29.8 -> 31.1 mm
- net ROW6: track 143.6 -> 144.6 mm
- net Net-(U1-Pad8): track 10.6 -> 11.6 mm
- net COL0: track 400.0 -> 400.9 mm
- net Net-(J1-Pad1): track 19.3 -> 20.2 mm
- net RESET: track 60.4 -> 61.2 mm
